File: KiCad/keyboard/keyboard.kicad_pcb (KiCad board)
At the start: 2 copper layers, 327.6 x 115.3 mm, 261 parts

Commit message: finishing led traces
Parts:
- removed D100, D101, D102, D103, D104, D105, D106, D107, D108, D109, D110, D111, D112, D113, D114, D115, D116, D117, D118, D119, D120, D121, D122, D123, D124, D125, D126, D127, D128, D129, D130, D131, D132, D133, D134, D135, D136, D137, D138, D139, D140, D141, D142, D143, D144, D145, D146, D147, D148, D149, D150, D151, D152, D153, D154, D155, D156, D157, D158, D159, D160, D161, D162, D163, D164, D165, D166, D167, D168, D169, D170, D171, D172, D173, D174, D88, D89, D90, D91, D92, D93, D94, D95, D96, D97, D98, D99: LED_RABG, keyboard_custom:RGB_LED_PLCC4-3.2x2.8mm_Reverse-Mount
- added C1: 100nF, Capacitor_SMD:C_0805_2012Metric, F.Cu at (24.0, -120.0)
- added C10: 100nF, Capacitor_SMD:C_0805_2012Metric, F.Cu at (229.0, -120.0)
- added C11: 100nF, Capacitor_SMD:C_0805_2012Metric, F.Cu at (258.0, -120.0)
- added C12: 100nF, Capacitor_SMD:C_0805_2012Metric, F.Cu at (277.0, -120.0)
- added C13: 100nF, Capacitor_SMD:C_0805_2012Metric, F.Cu at (296.0, -120.0)
- added C14: 100nF, Capacitor_SMD:C_0805_2012Metric, F.Cu at (315.0, -120.0)
- added C15: 100nF, Capacitor_SMD:C_0805_2012Metric, F.Cu at (334.0, -120.0)
- added C16: 100nF, Capacitor_SMD:C_0805_2012Metric, F.Cu at (24.0, -101.0)
- added C17: 100nF, Capacitor_SMD:C_0805_2012Metric, F.Cu at (48.0, -101.0)
- added C18: 100nF, Capacitor_SMD:C_0805_2012Metric, F.Cu at (67.0, -101.1)
- added C19: 100nF, Capacitor_SMD:C_0805_2012Metric, F.Cu at (86.0, -101.0)
- added C2: 100nF, Capacitor_SMD:C_0805_2012Metric, F.Cu at (48.0, -120.0)
- added C20: 100nF, Capacitor_SMD:C_0805_2012Metric, F.Cu at (105.0, -101.0)
- added C21: 100nF, Capacitor_SMD:C_0805_2012Metric, F.Cu at (124.0, -101.0)
- added C22: 100nF, Capacitor_SMD:C_0805_2012Metric, F.Cu at (143.0, -101.0)
- added C23: 100nF, Capacitor_SMD:C_0805_2012Metric, F.Cu at (163.0, -101.0)
- added C24: 100nF, Capacitor_SMD:C_0805_2012Metric, F.Cu at (182.0, -101.0)
- added C25: 100nF, Capacitor_SMD:C_0805_2012Metric, F.Cu at (201.0, -101.0)
- added C26: 100nF, Capacitor_SMD:C_0805_2012Metric, F.Cu at (220.0, -101.0)
- added C27: 100nF, Capacitor_SMD:C_0805_2012Metric, F.Cu at (239.0, -101.0)
- added C28: 100nF, Capacitor_SMD:C_0805_2012Metric, F.Cu at (258.0, -101.0)
- added C29: 100nF, Capacitor_SMD:C_0805_2012Metric, F.Cu at (277.0, -101.0)
- added C3: 100nF, Capacitor_SMD:C_0805_2012Metric, F.Cu at (86.0, -120.0)
- added C30: 100nF, Capacitor_SMD:C_0805_2012Metric, F.Cu at (305.0, -101.0)
- added C31: 100nF, Capacitor_SMD:C_0805_2012Metric, F.Cu at (334.0, -101.0)
- added C32: 100nF, Capacitor_SMD:C_0805_2012Metric, F.Cu at (23.8, -82.0)
- added C33: 100nF, Capacitor_SMD:C_0805_2012Metric, F.Cu at (52.4, -82.0)
- added C34: 100nF, Capacitor_SMD:C_0805_2012Metric, F.Cu at (76.2, -82.0)
- added C35: 100nF, Capacitor_SMD:C_0805_2012Metric, F.Cu at (95.2, -82.0)
- added C36: 100nF, Capacitor_SMD:C_0805_2012Metric, F.Cu at (114.3, -82.0)
- added C37: 100nF, Capacitor_SMD:C_0805_2012Metric, F.Cu at (133.3, -82.0)
- added C38: 100nF, Capacitor_SMD:C_0805_2012Metric, F.Cu at (152.4, -82.0)
- added C39: 100nF, Capacitor_SMD:C_0805_2012Metric, F.Cu at (171.4, -82.0)
- added C4: 100nF, Capacitor_SMD:C_0805_2012Metric, F.Cu at (105.0, -120.0)
- added C40: 100nF, Capacitor_SMD:C_0805_2012Metric, F.Cu at (190.5, -82.0)
- added C41: 100nF, Capacitor_SMD:C_0805_2012Metric, F.Cu at (209.6, -82.0)
- added C42: 100nF, Capacitor_SMD:C_0805_2012Metric, F.Cu at (228.6, -82.0)
- added C43: 100nF, Capacitor_SMD:C_0805_2012Metric, F.Cu at (247.7, -82.0)
- added C44: 100nF, Capacitor_SMD:C_0805_2012Metric, F.Cu at (266.7, -82.0)
- added C45: 100nF, Capacitor_SMD:C_0805_2012Metric, F.Cu at (285.8, -82.0)
- added C46: 100nF, Capacitor_SMD:C_0805_2012Metric, F.Cu at (309.6, -82.0)
- added C47: 100nF, Capacitor_SMD:C_0805_2012Metric, F.Cu at (333.4, -82.0)
- added C48: 100nF, Capacitor_SMD:C_0805_2012Metric, F.Cu at (23.8, -63.0)
- added C49: 100nF, Capacitor_SMD:C_0805_2012Metric, F.Cu at (54.8, -63.0)
- added C5: 100nF, Capacitor_SMD:C_0805_2012Metric, F.Cu at (124.0, -120.0)
- added C50: 100nF, Capacitor_SMD:C_0805_2012Metric, F.Cu at (81.0, -63.0)
- added C51: 100nF, Capacitor_SMD:C_0805_2012Metric, F.Cu at (100.0, -63.0)
- added C52: 100nF, Capacitor_SMD:C_0805_2012Metric, F.Cu at (119.1, -63.0)
- added C53: 100nF, Capacitor_SMD:C_0805_2012Metric, F.Cu at (138.1, -63.0)
- added C54: 100nF, Capacitor_SMD:C_0805_2012Metric, F.Cu at (157.2, -63.0)
- added C55: 100nF, Capacitor_SMD:C_0805_2012Metric, F.Cu at (176.2, -63.0)
- added C56: 100nF, Capacitor_SMD:C_0805_2012Metric, F.Cu at (195.3, -63.0)
- added C57: 100nF, Capacitor_SMD:C_0805_2012Metric, F.Cu at (214.3, -63.0)
- added C58: 100nF, Capacitor_SMD:C_0805_2012Metric, F.Cu at (233.4, -63.0)
- added C59: 100nF, Capacitor_SMD:C_0805_2012Metric, F.Cu at (252.4, -63.0)
- added C6: 100nF, Capacitor_SMD:C_0805_2012Metric, F.Cu at (143.0, -120.0)
- added C60: 100nF, Capacitor_SMD:C_0805_2012Metric, F.Cu at (271.5, -62.9)
- added C61: 100nF, Capacitor_SMD:C_0805_2012Metric, F.Cu at (302.4, -63.0)
- added C62: 100nF, Capacitor_SMD:C_0805_2012Metric, F.Cu at (333.4, -63.0)
- added C7: 100nF, Capacitor_SMD:C_0805_2012Metric, F.Cu at (172.0, -120.0)
- added C8: 100nF, Capacitor_SMD:C_0805_2012Metric, F.Cu at (191.0, -120.0)
- added C9: 100nF, Capacitor_SMD:C_0805_2012Metric, F.Cu at (210.0, -120.0)
- added LED1: WS2812B, keyboard_custom:WS2812B-2020, F.Cu at (19.1, -119.0)
- added LED10: WS2812B, keyboard_custom:WS2812B-2020, F.Cu at (50.0, -61.9)
- added LED13: WS2812B, keyboard_custom:WS2812B-2020, F.Cu at (61.9, -100.0)
- added LED14: WS2812B, keyboard_custom:WS2812B-2020, F.Cu at (71.4, -81.0)
- added LED15: WS2812B, keyboard_custom:WS2812B-2020, F.Cu at (76.2, -61.9)
- added LED18: WS2812B, keyboard_custom:WS2812B-2020, F.Cu at (81.0, -119.1)
- added LED19: WS2812B, keyboard_custom:WS2812B-2020, F.Cu at (81.0, -100.0)
- added LED2: WS2812B, keyboard_custom:WS2812B-2020, F.Cu at (19.1, -100.0)
- added LED20: WS2812B, keyboard_custom:WS2812B-2020, F.Cu at (90.5, -81.0)
- added LED21: WS2812B, keyboard_custom:WS2812B-2020, F.Cu at (95.2, -61.9)
- added LED24: WS2812B, keyboard_custom:WS2812B-2020, F.Cu at (100.0, -119.1)
- added LED25: WS2812B, keyboard_custom:WS2812B-2020, F.Cu at (100.0, -100.0)
- added LED26: WS2812B, keyboard_custom:WS2812B-2020, F.Cu at (109.5, -81.0)
- added LED27: WS2812B, keyboard_custom:WS2812B-2020, F.Cu at (114.3, -61.9)
- added LED29: WS2812B, keyboard_custom:WS2812B-2020, F.Cu at (119.1, -119.1)
- added LED3: WS2812B, keyboard_custom:WS2812B-2020, F.Cu at (19.1, -81.0)
- added LED30: WS2812B, keyboard_custom:WS2812B-2020, F.Cu at (119.1, -100.0)
- added LED31: WS2812B, keyboard_custom:WS2812B-2020, F.Cu at (128.6, -81.0)
- added LED32: WS2812B, keyboard_custom:WS2812B-2020, F.Cu at (133.3, -61.9)
- added LED34: WS2812B, keyboard_custom:WS2812B-2020, F.Cu at (138.1, -119.1)
- added LED35: WS2812B, keyboard_custom:WS2812B-2020, F.Cu at (138.1, -100.0)
- added LED36: WS2812B, keyboard_custom:WS2812B-2020, F.Cu at (147.6, -81.0)
- added LED37: WS2812B, keyboard_custom:WS2812B-2020, F.Cu at (152.4, -61.9)
- added LED4: WS2812B, keyboard_custom:WS2812B-2020, F.Cu at (19.1, -61.9)
- added LED40: WS2812B, keyboard_custom:WS2812B-2020, F.Cu at (166.7, -119.1)
- added LED41: WS2812B, keyboard_custom:WS2812B-2020, F.Cu at (157.2, -100.0)
- added LED42: WS2812B, keyboard_custom:WS2812B-2020, F.Cu at (166.7, -81.0)
- added LED43: WS2812B, keyboard_custom:WS2812B-2020, F.Cu at (171.4, -61.9)
- added LED45: WS2812B, keyboard_custom:WS2812B-2020, F.Cu at (185.7, -119.1)
- added LED46: WS2812B, keyboard_custom:WS2812B-2020, F.Cu at (176.2, -100.0)
- added LED47: WS2812B, keyboard_custom:WS2812B-2020, F.Cu at (185.7, -81.0)
- added LED48: WS2812B, keyboard_custom:WS2812B-2020, F.Cu at (190.5, -61.9)
- added LED50: WS2812B, keyboard_custom:WS2812B-2020, F.Cu at (204.8, -119.1)
- added LED51: WS2812B, keyboard_custom:WS2812B-2020, F.Cu at (195.3, -100.0)
- added LED52: WS2812B, keyboard_custom:WS2812B-2020, F.Cu at (204.8, -81.0)
- added LED53: WS2812B, keyboard_custom:WS2812B-2020, F.Cu at (209.6, -61.9)
- added LED55: WS2812B, keyboard_custom:WS2812B-2020, F.Cu at (223.8, -119.1)
- added LED56: WS2812B, keyboard_custom:WS2812B-2020, F.Cu at (214.3, -100.0)
- added LED57: WS2812B, keyboard_custom:WS2812B-2020, F.Cu at (223.8, -81.0)
- added LED58: WS2812B, keyboard_custom:WS2812B-2020, F.Cu at (228.6, -61.9)
- added LED61: WS2812B, keyboard_custom:WS2812B-2020, F.Cu at (252.4, -119.1)
- added LED62: WS2812B, keyboard_custom:WS2812B-2020, F.Cu at (233.4, -100.0)
- added LED63: WS2812B, keyboard_custom:WS2812B-2020, F.Cu at (242.9, -81.0)
- added LED64: WS2812B, keyboard_custom:WS2812B-2020, F.Cu at (247.7, -61.9)
- added LED67: WS2812B, keyboard_custom:WS2812B-2020, F.Cu at (271.5, -119.1)
- added LED68: WS2812B, keyboard_custom:WS2812B-2020, F.Cu at (252.4, -100.0)
- added LED69: WS2812B, keyboard_custom:WS2812B-2020, F.Cu at (261.9, -81.0)
- added LED7: WS2812B, keyboard_custom:WS2812B-2020, F.Cu at (42.9, -119.1)
- added LED70: WS2812B, keyboard_custom:WS2812B-2020, F.Cu at (266.7, -61.9)
- added LED73: WS2812B, keyboard_custom:WS2812B-2020, F.Cu at (290.5, -119.1)
- added LED74: WS2812B, keyboard_custom:WS2812B-2020, F.Cu at (271.5, -100.0)
- added LED75: WS2812B, keyboard_custom:WS2812B-2020, F.Cu at (281.0, -81.0)
- added LED76: WS2812B, keyboard_custom:WS2812B-2020, F.Cu at (297.7, -61.9)
- added LED79: WS2812B, keyboard_custom:WS2812B-2020, F.Cu at (309.6, -119.1)
- added LED8: WS2812B, keyboard_custom:WS2812B-2020, F.Cu at (42.9, -100.0)
- added LED80: WS2812B, keyboard_custom:WS2812B-2020, F.Cu at (300.0, -100.0)
- added LED81: WS2812B, keyboard_custom:WS2812B-2020, F.Cu at (304.8, -81.0)
- added LED82: WS2812B, keyboard_custom:WS2812B-2020, F.Cu at (328.6, -61.9)
- added LED85: WS2812B, keyboard_custom:WS2812B-2020, F.Cu at (328.6, -119.1)
- added LED86: WS2812B, keyboard_custom:WS2812B-2020, F.Cu at (328.6, -100.0)
- added LED87: WS2812B, keyboard_custom:WS2812B-2020, F.Cu at (328.6, -81.0)
- added LED9: WS2812B, keyboard_custom:WS2812B-2020, F.Cu at (47.6, -81.0)
- D1, D10, D11, D12, D13, D14, D15, D16, D17, D18, D19, D2, D20, D21, D22, D23, D24, D25, D26, D27, D28, D29, D3, D30, D31, D32, D33, D34, D35, D36, D37, D38, D39, D4, D40, D41, D42, D43, D44, D45, D46, D47, D48, D49, D5, D50, D51, D52, D53, D54, D55, D56, D57, D58, D59, D6, D60, D61, D62, D63, D64, D65, D66, D67, D68, D69, D7, D70, D71, D72, D73, D74, D75, D76, D77, D78, D79, D8, D80, D81, D82, D83, D84, D85, D86, D87, D9: moved to F.Cu
- MX', MX-_1, MX.>1, MX/?1, MX0, MX1, MX2, MX3, MX4, MX5, MX6, MX7, MX8, MX9, MX;:1, MX=+1, MXA1, MXB1, MXC1, MXD1, MXDEL1, MXDN1, MXE1, MXEND1, MXESC1, MXF1, MXF10, MXF11, MXF12, MXF13, MXF2, MXF3, MXF4, MXF5, MXF6, MXF7, MXF8, MXF9, MXG1, MXH1, MXHOME1, MXI1, MXJ1, MXK,<1, MXK1, MXL1, MXLFT1, MXM1, MXM2, MXM3, MXM4, MXM5, MXM6, MXM7, MXN1, MXO1, MXP1, MXPGDN1, MXPGUP1, MXQ1, MXR1, MXRT1, MXS1, MXT1, MXTILDE1, MXU1, MXUP1, MXV1, MXW1, MXX1, MXY1, MXZ1, MX[{1, MX]}1: footprint MX_Only:MXOnly-1U-Hotswap -> MX_Only:MXOnly-1U-NoLED
- MXBACK1: footprint MX_Only:MXOnly-2U-Hotswap-ReversedStabilizers -> MX_Only:MXOnly-2U-ReversedStabilizers-NoLED
- MXCAPS1, MXRSHFT1: footprint MX_Only:MXOnly-1.75U-Hotswap -> MX_Only:MXOnly-1.75U-NoLED
- MXFN1, MXLALT1, MXLCTL1, MXRALT1, MXWIN1: footprint MX_Only:MXOnly-1.25U-Hotswap -> MX_Only:MXOnly-1.25U-NoLED
- MXLSHFT1, MX\N1: footprint MX_Only:MXOnly-2.25U-Hotswap-ReversedStabilizers -> MX_Only:MXOnly-2.25U-ReversedStabilizers-NoLED
- MXSPACE1: footprint MX_Only:MXOnly-6.25U-Hotswap -> MX_Only:MXOnly-6.25U-NoLED
- MXTAB1, MX\|1: footprint MX_Only:MXOnly-1.5U-Hotswap -> MX_Only:MXOnly-1.5U-NoLED
- moved D84 12.8 mm to (330.9, -12.0), turned to 180 degrees
- moved D6 12.1 mm to (24.5, -11.8), turned to 0 degrees
- moved D67 11.7 mm to (279.0, -107.3), turned to 270 degrees
- moved D61 11.4 mm to (260.0, -107.7), turned to 270 degrees
- moved D73 11.4 mm to (298.0, -107.7), turned to 270 degrees
- moved D79 11.4 mm to (317.0, -107.7), turned to 270 degrees
- moved D40 11.4 mm to (174.0, -107.7), turned to 270 degrees
- moved D45 11.4 mm to (193.0, -107.7), turned to 270 degrees
- moved D50 11.4 mm to (212.0, -107.7), turned to 270 degrees
- moved D18 11.4 mm to (88.1, -107.7), turned to 270 degrees
- moved D24 11.4 mm to (107.2, -107.7), turned to 270 degrees
- moved D29 11.4 mm to (126.2, -107.7), turned to 270 degrees
- moved D34 11.4 mm to (145.3, -107.7), turned to 270 degrees
- moved D55 11.4 mm to (231.0, -107.7), turned to 270 degrees
- moved D7 11.4 mm to (50.0, -107.7), turned to 270 degrees
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Routing:
- net Net-(C1-Pad1): track 0.00 -> 1459.6 mm, vias 0 -> 4
- net GND: track 0.00 -> 1403.4 mm
- net Net-(LED3-Pad3): track 0.00 -> 347.7 mm, vias 0 -> 2
- net Net-(LED2-Pad3): track 0.00 -> 346.2 mm, vias 0 -> 2
- net Net-(LED4-Pad3): track 0.00 -> 345.0 mm, vias 0 -> 2
- net Net-(D11-Pad2): track 0.00 -> 314.8 mm
- net Net-(LED82-Pad1): track 0.00 -> 314.5 mm, vias 0 -> 1
- net Net-(D12-Pad2): track 0.00 -> 307.5 mm
- net Net-(MX'"1-Pad2): track 0.00 -> 124.6 mm
- net Net-(MX=+1-Pad2): track 0.00 -> 123.2 mm
- net Net-(MX/?1-Pad2): track 0.00 -> 119.5 mm
- net Net-(MXBACK1-Pad2): track 0.00 -> 115.2 mm
- net Net-(MX2-Pad2): track 0.00 -> 113.5 mm
- net Net-(MX.>1-Pad2): track 0.00 -> 110.0 mm
- net Net-(MX5-Pad2): track 0.00 -> 106.1 mm
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
Commit message: pcb almost finished, BOM generated
Parts:
- removed C1, C10, C11, C12, C13, C14, C15, C16, C17, C18, C19, C2, C20, C21, C22, C23, C24, C25, C26, C27, C28, C29, C3, C30, C31, C4, C5, C6, C7, C8, C9: 100nF, Capacitor_SMD:C_0805_2012Metric
- removed D1, D10, D11, D12, D13, D14, D15, D16, D17, D18, D19, D2, D20, D21, D22, D23, D24, D25, D26, D27, D28, D29, D3, D30, D31, D32, D33, D34, D35, D36, D37, D38, D39, D4, D40, D41, D42, D43, D44, D45, D46, D47, D48, D49, D5, D50, D51, D52, D53, D54, D55, D56, D57, D58, D59, D6, D60, D61, D62, D63, D64, D65, D66, D67, D68, D69, D7, D70, D71, D72, D73, D74, D75, D76, D77, D78, D79, D8, D80, D81, D82, D83, D84, D85, D86, D87, D9: DIODE, Diode_SMD:D_SOD-123
- removed LED1, LED13, LED18, LED19, LED2, LED24, LED25, LED29, LED30, LED34, LED35, LED40, LED41, LED45, LED46, LED50, LED51, LED55, LED56, LED61, LED62, LED67, LED68, LED7, LED73, LED74, LED79, LED8, LED80, LED85, LED86: WS2812B, keyboard_custom:WS2812B-2020
- removed MX0, MX1, MX2, MX4, MX7, MX9: MX-LED, MX_Only:MXOnly-1U-NoLED
- added C63: 100nF, Capacitor_SMD:C_0805_2012Metric, F.Cu at (23.8, -44.0)
- added C64: 100nF, Capacitor_SMD:C_0805_2012Metric, F.Cu at (59.5, -44.0)
- added C65: 100nF, Capacitor_SMD:C_0805_2012Metric, F.Cu at (90.5, -44.0)
- added C66: 100nF, Capacitor_SMD:C_0805_2012Metric, F.Cu at (109.5, -44.0)
- added C67: 100nF, Capacitor_SMD:C_0805_2012Metric, F.Cu at (128.6, -44.0)
- added C68: 100nF, Capacitor_SMD:C_0805_2012Metric, F.Cu at (147.6, -44.0)
- added C69: 100nF, Capacitor_SMD:C_0805_2012Metric, F.Cu at (166.7, -44.0)
- added C70: 100nF, Capacitor_SMD:C_0805_2012Metric, F.Cu at (185.7, -44.0)
- added C71: 100nF, Capacitor_SMD:C_0805_2012Metric, F.Cu at (204.8, -44.0)
- added C72: 100nF, Capacitor_SMD:C_0805_2012Metric, F.Cu at (223.8, -44.0)
- added C73: 100nF, Capacitor_SMD:C_0805_2012Metric, F.Cu at (242.9, -44.0)
- added C74: 100nF, Capacitor_SMD:C_0805_2012Metric, F.Cu at (261.9, -44.0)
- added C75: 100nF, Capacitor_SMD:C_0805_2012Metric, F.Cu at (288.1, -44.0)
- added C76: 100nF, Capacitor_SMD:C_0805_2012Metric, F.Cu at (314.3, -44.0)
- added C77: 100nF, Capacitor_SMD:C_0805_2012Metric, F.Cu at (333.4, -44.0)
- added C78: 100nF, Capacitor_SMD:C_0805_2012Metric, F.Cu at (23.8, -25.0)
- added C79: 100nF, Capacitor_SMD:C_0805_2012Metric, F.Cu at (50.0, -25.0)
- added C80: 100nF, Capacitor_SMD:C_0805_2012Metric, F.Cu at (73.8, -25.0)
- added C81: 100nF, Capacitor_SMD:C_0805_2012Metric, F.Cu at (97.6, -25.0)
- added C82: 100nF, Capacitor_SMD:C_0805_2012Metric, F.Cu at (169.1, -25.0)
- added C83: 100nF, Capacitor_SMD:C_0805_2012Metric, F.Cu at (240.5, -25.0)
- added C84: 100nF, Capacitor_SMD:C_0805_2012Metric, F.Cu at (264.3, -25.0)
- added C85: 100nF, Capacitor_SMD:C_0805_2012Metric, F.Cu at (295.3, -25.0)
- added C86: 100nF, Capacitor_SMD:C_0805_2012Metric, F.Cu at (314.3, -25.0)
- added C87: 100nF, Capacitor_SMD:C_0805_2012Metric, F.Cu at (333.4, -25.0)
- added C88: 100nF, Capacitor_SMD:C_0603_1608Metric, B.Cu at (61.8, -106.8)
- added C89: 100nF, Capacitor_SMD:C_0603_1608Metric, B.Cu at (68.0, -106.8)
- added C90: 100nF, Capacitor_SMD:C_0603_1608Metric, B.Cu at (57.2, -109.0)
- added C91: 100nF, Capacitor_SMD:C_0603_1608Metric, B.Cu at (62.8, -118.8)
- added C92: 10uF, Capacitor_SMD:C_0603_1608Metric, B.Cu at (70.0, -115.5)
- added C93: 1uF, Capacitor_SMD:C_0603_1608Metric, B.Cu at (57.0, -112.2)
- added C94: 22pF, Capacitor_SMD:C_0603_1608Metric, B.Cu at (51.2, -120.7)
- added C95: 22pF, Capacitor_SMD:C_0603_1608Metric, B.Cu at (57.1, -120.7)
- added C96: 10uF, Capacitor_SMD:C_0603_1608Metric, B.Cu at (60.5, -120.5)
- added D88: PRTR5V0U2X, Package_TO_SOT_SMD:SOT-143, B.Cu at (31.0, -110.5)
- added F1: 6A, Fuse:Fuse_0805_2012Metric, B.Cu at (27.2, -115.0)
- added FB1: 60Ω@100MHz, 3A, keyboard_custom:Ferrite_SMD_0603, B.Cu at (37.0, -118.8)
- added LED11: WS2812B, keyboard_custom:WS2812B-2020, F.Cu at (54.8, -43.0)
- added LED12: WS2812B, keyboard_custom:WS2812B-2020, F.Cu at (45.2, -24.0)
- added LED16: WS2812B, keyboard_custom:WS2812B-2020, F.Cu at (85.7, -43.0)
- added LED17: WS2812B, keyboard_custom:WS2812B-2020, F.Cu at (69.1, -24.0)
- added LED22: WS2812B, keyboard_custom:WS2812B-2020, F.Cu at (104.8, -43.0)
- added LED23: WS2812B, keyboard_custom:WS2812B-2020, F.Cu at (92.9, -24.0)
- added LED28: WS2812B, keyboard_custom:WS2812B-2020, F.Cu at (123.8, -43.0)
- added LED33: WS2812B, keyboard_custom:WS2812B-2020, F.Cu at (142.9, -43.0)
- added LED38: WS2812B, keyboard_custom:WS2812B-2020, F.Cu at (161.9, -43.0)
- added LED39: WS2812B, keyboard_custom:WS2812B-2020, F.Cu at (164.3, -24.0)
- added LED44: WS2812B, keyboard_custom:WS2812B-2020, F.Cu at (181.0, -43.0)
- added LED49: WS2812B, keyboard_custom:WS2812B-2020, F.Cu at (200.0, -43.0)
- added LED5: WS2812B, keyboard_custom:WS2812B-2020, F.Cu at (19.1, -43.0)
- added LED54: WS2812B, keyboard_custom:WS2812B-2020, F.Cu at (219.1, -43.0)
- added LED59: WS2812B, keyboard_custom:WS2812B-2020, F.Cu at (238.1, -43.0)
- added LED6: WS2812B, keyboard_custom:WS2812B-2020, F.Cu at (19.1, -24.0)
- added LED60: WS2812B, keyboard_custom:WS2812B-2020, F.Cu at (235.7, -24.0)
- added LED65: WS2812B, keyboard_custom:WS2812B-2020, F.Cu at (257.2, -43.0)
- added LED66: WS2812B, keyboard_custom:WS2812B-2020, F.Cu at (259.6, -24.0)
- added LED71: WS2812B, keyboard_custom:WS2812B-2020, F.Cu at (283.4, -43.1)
- added LED72: WS2812B, keyboard_custom:WS2812B-2020, F.Cu at (290.5, -24.0)
- added LED77: WS2812B, keyboard_custom:WS2812B-2020, F.Cu at (309.6, -43.0)
- added LED78: WS2812B, keyboard_custom:WS2812B-2020, F.Cu at (309.6, -24.0)
- added LED83: WS2812B, keyboard_custom:WS2812B-2020, F.Cu at (328.6, -43.0)
- added LED84: WS2812B, keyboard_custom:WS2812B-2020, F.Cu at (328.6, -24.0)
- added R1: 5.1kΩ, Resistor_SMD:R_0805_2012Metric, B.Cu at (29.5, -115.0)
- added R2: 5.1kΩ, Resistor_SMD:R_0805_2012Metric, B.Cu at (33.8, -115.8)
- added R3: 22Ω, Resistor_SMD:R_0805_2012Metric, B.Cu at (53.2, -111.2)
- added R4: 22Ω, Resistor_SMD:R_0805_2012Metric, B.Cu at (53.2, -109.0)
- added R5: 10kΩ, Resistor_SMD:R_0805_2012Metric, B.Cu at (60.2, -118.2)
- added R6: 10kΩ, Resistor_SMD:R_0805_2012Metric, B.Cu at (72.5, -108.5)
- added SW1: SW_Push, Button_Switch_SMD:Panasonic_EVQPUM_EVQPUD, B.Cu at (41.5, -120.5)
- added U1: ATmega32U4-MU, Package_DFN_QFN:QFN-44-1EP_7x7mm_P0.5mm_EP5.2x5.2mm, B.Cu at (64.8, -112.0)
- added USB1: USB_C_Receptacle_USB2.0, Connector_USB:USB_C_Receptacle_HRO_TYPE-C-31-M-12, B.Cu at (31.0, -123.0)
- added X1: 16MHz, Crystal:Crystal_SMD_3225-4Pin_3.2x2.5mm, B.Cu at (54.2, -120.5)
Connections:
- net Net-(MX'"1-Pad2) renamed Col12
- net Net-(MX.>1-Pad2) renamed Col10
- net Net-(MX/?1-Pad2) renamed Col11
- net Net-(MX1-Pad2) renamed Col2
- net Net-(MX2-Pad2) renamed Col3
- net Net-(MX3-Pad2) renamed Col4
- net Net-(MX4-Pad2) renamed Col5
- net Net-(MX5-Pad2) renamed Col6
- net Net-(MX6-Pad2) renamed Col7
- net Net-(MX7-Pad2) renamed Col8
- net Net-(MX8-Pad2) renamed Col9
- net Net-(MX=+1-Pad2) renamed Col13
- net Net-(MXBACK1-Pad2) renamed Col14
- net Net-(MXCAPS1-Pad2) renamed Col1
- net Net-(MXDEL1-Pad2) renamed Col15
- net Net-(MXM1-Pad2) renamed Col0
Routing:
- net Net-(C1-Pad1): track 1459.6 -> 0.00 mm, vias 4 -> 0
- net GND: track 1403.4 -> 0.00 mm
- net Net-(LED3-Pad3): track 347.7 -> 0.00 mm, vias 2 -> 0
- net Net-(LED2-Pad3): track 346.2 -> 0.00 mm, vias 2 -> 0
- net Net-(LED4-Pad3): track 345.0 -> 0.00 mm, vias 2 -> 0
- net Net-(D11-Pad2): track 314.8 -> 0.00 mm
- net Net-(D10-Pad2): track 314.8 -> 0.00 mm
- net Net-(LED5-Pad3): track 314.5 -> 0.00 mm, vias 1 -> 0
- net Net-(D13-Pad2): track 314.2 -> 0.00 mm
- net Net-(D1-Pad2): track 309.5 -> 0.00 mm
- net Net-(D14-Pad2): track 309.0 -> 0.00 mm
- net Net-(D12-Pad2): track 307.5 -> 0.00 mm
- net Col12: track 124.6 -> 0.00 mm
- net Col13: track 123.2 -> 0.00 mm
- net Col11: track 119.5 -> 0.00 mm
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Other:
- board outline removed
- net class Power added: clearance 0.2, trace_width 0.381, via_dia 0.8, via_drill 0.4

Commit message: added 6pin ISP to load bootloader
Parts:
- added J1: AVR-ISP-6, keyboard_custom:AVR-ISP-6, F.Cu at (13.2, -103.2)
- added REF**: MountingHole_3.5mm, MountingHole:MountingHole_3.5mm, F.Cu at (296.5, -36.0)
- added REF**: MountingHole_3.5mm, MountingHole:MountingHole_3.5mm, F.Cu at (193.5, -17.1)
- added REF**: MountingHole_3.5mm, MountingHole:MountingHole_3.5mm, F.Cu at (140.2, -17.0)
- added REF**: MountingHole_3.5mm, MountingHole:MountingHole_3.5mm, F.Cu at (33.4, -35.7)
- added REF**: MountingHole_3.5mm, MountingHole:MountingHole_3.5mm, F.Cu at (31.8, -92.8)
- added REF**: MountingHole_3.5mm, MountingHole:MountingHole_3.5mm, F.Cu at (239.2, -111.4)
- added REF**: MountingHole_3.5mm, MountingHole:MountingHole_3.5mm, F.Cu at (317.8, -74.0)
- added REF**: MountingHole_3.5mm, MountingHole:MountingHole_3.5mm, F.Cu at (153.5, -111.4)
- F1: value 6A -> 1A hold, 2A trip
- FB1: value 60Ω@100MHz, 3A -> 60Ω@100MHz, 1A
Other:
- net class Power removed
