File: KiCad/keyboard/keyboard.sch (KiCad schematic (older format))
At the start: 262 parts

Commit message: finishing led traces
Parts:
- removed D100, D101, D102, D103, D104, D105, D106, D107, D108, D109, D110, D111, D112, D113, D114, D115, D116, D117, D118, D119, D120, D121, D122, D123, D124, D125, D126, D127, D128, D129, D130, D131, D132, D133, D134, D135, D136, D137, D138, D139, D140, D141, D142, D143, D144, D145, D146, D147, D148, D149, D150, D151, D152, D153, D154, D155, D156, D157, D158, D159, D160, D161, D162, D163, D164, D165, D166, D167, D168, D169, D170, D171, D172, D173, D174, D88, D89, D90, D91, D92, D93, D94, D95, D96, D97, D98, D99: LED_RABG, keyboard_custom:RGB_LED_PLCC4-3.2x2.8mm_Reverse-Mount, symbol Device:LED_RABG
- removed MCU?: STM32Wb55Rx-VQFPN68, symbol Keyboard_Custom:STM32Wb55Rx-VQFPN68
- added C1, C10, C11, C12, C13, C14, C15, C16, C17, C18, C19, C2, C20, C21, C22, C23, C24, C25, C26, C27, C28, C29, C3, C30, C31, C32, C33, C34, C35, C36, C37, C38, C39, C4, C40, C41, C42, C43, C44, C45, C46, C47, C48, C49, C5, C50, C51, C52, C53, C54, C55, C56, C57, C58, C59, C6, C60, C61, C62, C7, C8, C9: 100nF, Capacitor_SMD:C_0805_2012Metric, symbol Device:C_Small
- added LED1, LED10, LED13, LED14, LED15, LED18, LED19, LED2, LED20, LED21, LED24, LED25, LED26, LED27, LED29, LED3, LED30, LED31, LED32, LED34, LED35, LED36, LED37, LED4, LED40, LED41, LED42, LED43, LED45, LED46, LED47, LED48, LED50, LED51, LED52, LED53, LED55, LED56, LED57, LED58, LED61, LED62, LED63, LED64, LED67, LED68, LED69, LED7, LED70, LED73, LED74, LED75, LED76, LED79, LED8, LED80, LED81, LED82, LED85, LED86, LED87, LED9: WS2812B, keyboard_custom:WS2812B-2020, symbol Keyboard_Custom:WS2812B
- MX'"1, MX-_1, MX.>1, MX/?1, MX0, MX1, MX2, MX3, MX4, MX5, MX6, MX7, MX8, MX9, MX;:1, MX=+1, MXA1, MXB1, MXC1, MXD1, MXDEL1, MXDN1, MXE1, MXEND1, MXESC1, MXF1, MXF10, MXF11, MXF12, MXF13, MXF2, MXF3, MXF4, MXF5, MXF6, MXF7, MXF8, MXF9, MXG1, MXH1, MXHOME1, MXI1, MXJ1, MXK,<1, MXK1, MXL1, MXLFT1, MXM1, MXM2, MXM3, MXM4, MXM5, MXM6, MXM7, MXN1, MXO1, MXP1, MXPGDN1, MXPGUP1, MXQ1, MXR1, MXRT1, MXS1, MXT1, MXTILDE1, MXU1, MXUP1, MXV1, MXW1, MXX1, MXY1, MXZ1, MX[{1, MX]}1: footprint MX_Only:MXOnly-1U-Hotswap -> MX_Only:MXOnly-1U-NoLED
- MXBACK1: footprint MX_Only:MXOnly-2U-Hotswap-ReversedStabilizers -> MX_Only:MXOnly-2U-ReversedStabilizers-NoLED
- MXCAPS1, MXRSHFT1: footprint MX_Only:MXOnly-1.75U-Hotswap -> MX_Only:MXOnly-1.75U-NoLED
- MXFN1, MXLALT1, MXLCTL1, MXRALT1, MXWIN1: footprint MX_Only:MXOnly-1.25U-Hotswap -> MX_Only:MXOnly-1.25U-NoLED
- MXLSHFT1, MX\N1: footprint MX_Only:MXOnly-2.25U-Hotswap-ReversedStabilizers -> MX_Only:MXOnly-2.25U-ReversedStabilizers-NoLED
- MXSPACE1: footprint MX_Only:MXOnly-6.25U-Hotswap -> MX_Only:MXOnly-6.25U-NoLED
- MXTAB1, MX\|1: footprint MX_Only:MXOnly-1.5U-Hotswap -> MX_Only:MXOnly-1.5U-NoLED
Connections:
- net labels added: GND
- wire segments 435 -> 1042

Commit message: pcb almost finished, BOM generated
Parts:
- added C63, C64, C65, C66, C67, C68, C69, C70, C71, C72, C73, C74, C75, C76, C77, C78, C79, C80, C81, C82, C83, C84, C85, C86, C87: 100nF, Capacitor_SMD:C_0805_2012Metric, symbol Device:C_Small
- added C88, C89, C90, C91: 100nF, Capacitor_SMD:C_0603_1608Metric, symbol Device:C_Small
- added C92, C96: 10uF, Capacitor_SMD:C_0603_1608Metric, symbol Device:C_Small
- added C93: 1uF, Capacitor_SMD:C_0603_1608Metric, symbol Device:C_Small
- added C94, C95: 22pF, Capacitor_SMD:C_0603_1608Metric, symbol Device:C_Small
- added D88: PRTR5V0U2X, Package_TO_SOT_SMD:SOT-143, symbol Power_Protection:PRTR5V0U2X
- added F1: 1A hold, 2A trip, Fuse:Fuse_0805_2012Metric, symbol Device:Polyfuse_Small
- added FB1: 60Ω@100MHz, 1A, keyboard_custom:Ferrite_SMD_0603, symbol Device:Ferrite_Bead_Small
- added LED11, LED12, LED16, LED17, LED22, LED23, LED28, LED33, LED38, LED39, LED44, LED49, LED5, LED54, LED59, LED6, LED60, LED65, LED66, LED71, LED72, LED77, LED78, LED83, LED84: WS2812B, keyboard_custom:WS2812B-2020, symbol Keyboard_Custom:WS2812B
- added R1, R2: 5.1kΩ, Resistor_SMD:R_0805_2012Metric, symbol Device:R_US
- added R3, R4: 22Ω, Resistor_SMD:R_0805_2012Metric, symbol Device:R_US
- added R5, R6: 10kΩ, Resistor_SMD:R_0805_2012Metric, symbol Device:R_US
- added SW1: SW_Push, Button_Switch_SMD:Panasonic_EVQPUM_EVQPUD, symbol Switch:SW_Push
- added U1: ATmega32U4-MU, Package_DFN_QFN:QFN-44-1EP_7x7mm_P0.5mm_EP5.2x5.2mm, symbol MCU_Microchip_ATmega:ATmega32U4-MU
- added USB1: USB_C_Receptacle_USB2.0, Connector_USB:USB_C_Receptacle_HRO_TYPE-C-31-M-12, symbol Connector:USB_C_Receptacle_USB2.0
- added X1: 16MHz, Crystal:Crystal_SMD_3225-4Pin_3.2x2.5mm, symbol Device:Crystal_GND24_Small
Connections:
- net GND: now also C63.2, C64.2, C65.2, C66.2, C67.2, C68.2, C69.2, C70.2, C71.2, C72.2, C73.2, C74.2, C75.2, C76.2, C77.2, C78.2, C79.2, C80.2, C81.2, C82.2, C83.2, C84.2, C85.2, C86.2, C87.2, C88.2, C89.2, C90.2, C91.2, C92.2, C93.2, C94.1, C95.1, C96.1, D88.1 (GND), FB1.1, LED11.2 (GND), LED12.2 (GND), LED16.2 (GND), LED17.2 (GND), LED22.2 (GND), LED23.2 (GND), LED28.2 (GND), LED33.2 (GND), LED38.2 (GND), LED39.2 (GND), LED44.2 (GND), LED49.2 (GND), LED5.2 (GND), LED54.2 (GND), LED59.2 (GND), LED6.2 (GND), LED60.2 (GND), LED65.2 (GND), LED66.2 (GND), LED71.2 (GND), LED72.2 (GND), LED77.2 (GND), LED78.2 (GND), LED83.2 (GND), LED84.2 (GND), R1.1, R2.1, R6.1, SW1.1, U1.15 (GND), U1.23 (GND), U1.35 (GND), U1.43 (GND), U1.45 (GND), U1.5 (UGND), USB1.A1 (GND), USB1.A12 (GND), USB1.B1 (GND), USB1.B12 (GND), X1.2, X1.4
- net Col0: now reaches MXM1.2 (ROW), MXM2.2 (ROW), MXM3.2 (ROW), MXM4.2 (ROW), MXM5.2 (ROW), MXM6.2 (ROW)
- net Col0: now also U1.10 (PB2)
- net Col1: now reaches MXCAPS1.2 (ROW), MXESC1.2 (ROW), MXLCTL1.2 (ROW), MXLSHFT1.2 (ROW), MXTAB1.2 (ROW), MXTILDE1.2 (ROW)
- net Col1: now also U1.9 (PB1)
- net Col3: now reaches MX2.2 (ROW), MXF1.2 (ROW), MXLALT1.2 (ROW), MXS1.2 (ROW), MXW1.2 (ROW), MXX1.2 (ROW)
- net Col3: now also U1.32 (PC7)
- net Col4: now reaches MX3.2 (ROW), MXC1.2 (ROW), MXD1.2 (ROW), MXE1.2 (ROW), MXF2.2 (ROW)
- net Col4: now also U1.31 (PC6)
- net Col5: now reaches MX4.2 (ROW), MXF3.2 (ROW), MXF4.2 (ROW), MXR1.2 (ROW), MXV1.2 (ROW)
- net Col5: now also U1.30 (PB6)
- net Col6: now reaches MX5.2 (ROW), MXB1.2 (ROW), MXF5.2 (ROW), MXG1.2 (ROW), MXSPACE1.2 (ROW), MXT1.2 (ROW)
- net Col6: now also U1.29 (PB5)
- net Col7: now reaches MX6.2 (ROW), MXF6.2 (ROW), MXH1.2 (ROW), MXN1.2 (ROW), MXY1.2 (ROW)
- net Col7: now also U1.28 (PB4)
- net Col8: now reaches MX7.2 (ROW), MXF7.2 (ROW), MXJ1.2 (ROW), MXM7.2 (ROW), MXU1.2 (ROW)
- net Col8: now also U1.27 (PD7)
- net Col9: now reaches MX8.2 (ROW), MXF8.2 (ROW), MXI1.2 (ROW), MXK,<1.2 (ROW), MXK1.2 (ROW)
- net Col9: now also U1.26 (PD6)
- net Col10: now reaches MX.>1.2 (ROW), MX9.2 (ROW), MXF9.2 (ROW), MXL1.2 (ROW), MXO1.2 (ROW), MXRALT1.2 (ROW)
- net Col10: now also U1.25 (PD4)
- net Col11: now reaches MX/?1.2 (ROW), MX0.2 (ROW), MX;:1.2 (ROW), MXF10.2 (ROW), MXFN1.2 (ROW), MXP1.2 (ROW)
- net Col11: now also U1.22 (PD5)
- net Col12: now reaches MX'"1.2 (ROW), MX-_1.2 (ROW), MXF11.2 (ROW), MXLFT1.2 (ROW), MXRSHFT1.2 (ROW), MX[{1.2 (ROW)
- net Col12: now also U1.21 (PD3)
- net Col13: now reaches MX=+1.2 (ROW), MXDN1.2 (ROW), MXF12.2 (ROW), MXUP1.2 (ROW), MX\N1.2 (ROW), MX]}1.2 (ROW)
- net Col13: now also U1.20 (PD2)
- net Col14: now reaches MXBACK1.2 (ROW), MXF13.2 (ROW), MXPGDN1.2 (ROW), MXPGUP1.2 (ROW), MXRT1.2 (ROW), MX\|1.2 (ROW)
- net Col14: now also U1.19 (PD1)
- net Col15: now reaches MXDEL1.2 (ROW), MXEND1.2 (ROW), MXHOME1.2 (ROW)
- net Col15: now also U1.18 (PD0)
- net Col2: now reaches MX1.2 (ROW), MXA1.2 (ROW), MXQ1.2 (ROW), MXWIN1.2 (ROW), MXZ1.2 (ROW)
- net Col2: now also U1.41 (PF0)
- net LEDIN: now reaches LED1.3 (DIN)
- net LEDIN: now also U1.11 (PB3)
- net at C1.1, C10.1, C11.1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: now also C63.1, C64.1, C65.1, C66.1, C67.1, C68.1, C69.1, C70.1, C71.1, C72.1, C73.1, C74.1, C75.1, C76.1, C77.1, C78.1, C79.1, C80.1, C81.1, C82.1, C83.1, C84.1, C85.1, C86.1, C87.1, LED11.4 (VDD), LED12.4 (VDD), LED16.4 (VDD), LED17.4 (VDD), LED22.4 (VDD), LED23.4 (VDD), LED28.4 (VDD), LED33.4 (VDD), LED38.4 (VDD), LED39.4 (VDD), LED44.4 (VDD), LED49.4 (VDD), LED5.4 (VDD), LED54.4 (VDD), LED59.4 (VDD), LED6.4 (VDD), LED60.4 (VDD), LED65.4 (VDD), LED66.4 (VDD), LED71.4 (VDD), LED72.4 (VDD), LED77.4 (VDD), LED78.4 (VDD), LED83.4 (VDD), LED84.4 (VDD)
- net Row0: now reaches D1.2 (A), D18.2 (A), D24.2 (A), D29.2 (A), D34.2 (A), D40.2 (A), D45.2 (A), D50.2 (A), D55.2 (A), D61.2 (A), D67.2 (A), D7.2 (A), D73.2 (A), D79.2 (A), D85.2 (A)
- net Row0: now also U1.1 (PE6)
- net Row1: now reaches D13.2 (A), D19.2 (A), D2.2 (A), D25.2 (A), D30.2 (A), D35.2 (A), D41.2 (A), D46.2 (A), D51.2 (A), D56.2 (A), D62.2 (A), D68.2 (A), D74.2 (A), D8.2 (A), D80.2 (A), D86.2 (A)
- net Row1: now also U1.40 (PF1)
- net Row2: now reaches D14.2 (A), D20.2 (A), D26.2 (A), D3.2 (A), D31.2 (A), D36.2 (A), D42.2 (A), D47.2 (A), D52.2 (A), D57.2 (A), D63.2 (A), D69.2 (A), D75.2 (A), D81.2 (A), D87.2 (A), D9.2 (A)
- net Row2: now also U1.39 (PF4)
- net Row3: now reaches D10.2 (A), D15.2 (A), D21.2 (A), D27.2 (A), D32.2 (A), D37.2 (A), D4.2 (A), D43.2 (A), D48.2 (A), D53.2 (A), D58.2 (A), D64.2 (A), D70.2 (A), D76.2 (A), D82.2 (A)
- net Row3: now also U1.38 (PF5)
- net Row4: now reaches D11.2 (A), D16.2 (A), D22.2 (A), D28.2 (A), D33.2 (A), D38.2 (A), D44.2 (A), D49.2 (A), D5.2 (A), D54.2 (A), D59.2 (A), D65.2 (A), D71.2 (A), D77.2 (A), D83.2 (A)
- net Row4: now also U1.37 (PF6)
- net Row5: now reaches D12.2 (A), D17.2 (A), D23.2 (A), D39.2 (A), D6.2 (A), D60.2 (A), D66.2 (A), D72.2 (A), D78.2 (A), D84.2 (A)
- net Row5: now also U1.36 (PF7)
- net at LED82.1 (DOUT): now also LED5.3 (DIN)
- new net: LED11.3 (DIN), LED5.1 (DOUT)
- new net: LED22.1 (DOUT), LED28.3 (DIN)
- new net: LED16.1 (DOUT), LED22.3 (DIN)
- new net: LED28.1 (DOUT), LED33.3 (DIN)
- new net: LED33.1 (DOUT), LED38.3 (DIN)
- new net: LED38.1 (DOUT), LED44.3 (DIN)
- new net: LED44.1 (DOUT), LED49.3 (DIN)
- new net: LED49.1 (DOUT), LED54.3 (DIN)
- new net: LED54.1 (DOUT), LED59.3 (DIN)
- new net: LED59.1 (DOUT), LED65.3 (DIN)
- new net: LED65.1 (DOUT), LED71.3 (DIN)
- new net: LED71.1 (DOUT), LED77.3 (DIN)
- new net: LED77.1 (DOUT), LED83.3 (DIN)
- new net: LED6.3 (DIN), LED83.1 (DOUT)
- new net: LED11.1 (DOUT), LED16.3 (DIN)
- new net: LED12.3 (DIN), LED6.1 (DOUT)
- new net: LED23.1 (DOUT), LED39.3 (DIN)
- new net: LED17.1 (DOUT), LED23.3 (DIN)
- new net: LED39.1 (DOUT), LED60.3 (DIN)
- new net: LED60.1 (DOUT), LED66.3 (DIN)
- new net: LED66.1 (DOUT), LED72.3 (DIN)
- new net: LED72.1 (DOUT), LED78.3 (DIN)
- new net: LED78.1 (DOUT), LED84.3 (DIN)
- new net: LED12.1 (DOUT), LED17.3 (DIN)
- new net: R4.1, U1.3 (D-)
- new net: R6.2, U1.33 (~HWB~/PE2)
- new net: R3.1, U1.4 (D+)
- new net: C93.1, U1.6 (UCAP)
- new net: FB1.2, USB1.S1 (SHIELD)
- new net: R1.2, USB1.A5 (CC1)
- new net: R2.2, USB1.B5 (CC2)
- new net: F1.2, USB1.A4 (VBUS), USB1.A9 (VBUS), USB1.B4 (VBUS), USB1.B9 (VBUS)
- new net +5V: C88.1, C89.1, C90.1, C91.1, C92.1, D88.4 (VCC), F1.1, R5.1, U1.14 (VCC), U1.2 (UVCC), U1.24 (AVCC), U1.34 (VCC), U1.44 (AVCC), U1.7 (VBUS)
- new net D+: D88.3 (I/O2), R3.2, USB1.A6 (D+), USB1.B6 (D+)
- new net D-: D88.2 (I/O1), R4.2, USB1.A7 (D-), USB1.B7 (D-)
- new net Reset: C96.2, R5.2, SW1.2, U1.13 (~RESET)
- new net XTAL1: C94.2, U1.17 (XTAL1), X1.1
- new net XTAL2: C95.2, U1.16 (XTAL2), X1.3
Other:
- moved on the sheet: C1, C10, C11, C12, C13, C14, C15, C16, C17, C18, C19, C2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

Commit message: added 6pin ISP to load bootloader
Parts:
- added J1: AVR-ISP-6, keyboard_custom:AVR-ISP-6, symbol Connector:AVR-ISP-6
- USB1: symbol Connector:USB_C_Receptacle_USB2.0 -> keyboard-rescue:USB_C_Receptacle_USB2.0-Connector
Connections:
- net +5V: now also J1.2 (VCC)
- net Col0: now also J1.1 (MISO)
- net Col1: now also J1.3 (SCK)
- net GND: now also J1.6 (GND)
- net LEDIN: now also J1.4 (MOSI)
- net Reset: now also J1.5 (~RST)
Other:
- moved on the sheet: C88, C89, C90, C91, C92, C94, C95, C96, D88, F1, FB1, R1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
